File: pcb/wearable_v2.kicad_sch (KiCad schematic)
At the start: 64 parts, among them J1 TYPE-C-31-M-12, Q1 AO3401A, U1 ESP32-C3-MINI-1-N4, U10 SHT40-AD1B-R3, U2 USBLC6-2SC6, U3 TP4054-42-SOT25R, U4 ME6211C33M5G-N, U5 XC6206P182MR, U6 TPS61099DRVR, U7 MAX30101EFD+T, U8 TMP117AIDRVR, U9 LSM6DS3TR-C

Commit message: Rename pcb_v2/ to pcb/ and confirm the inductor's ratings with the vendor
Folder, footprint library nickname, 3D-model directory and every reference
across CLAUDE.md, parts/ and the project files now use "pcb". The KiCad
project files keep the wearable_v2 name: that "v2" identifies the board
revision, not the folder scheme, and renaming it would mean rewriting the
project name embedded in every symbol instance path.

Note for anyone reading history: an unrelated abandoned pcb/ folder was
deleted on 2026-09-14 (recoverable at ebf99dc), so `git log -- pcb/` spans
two different things.

MAKK2016T2R2M ratings are now manufacturer-confirmed rather than taken from
a distributor listing: 2.2uH +/-20%, Isat 1.5A, Irms 1.5A, DCR 0.16 ohm max,
2.0 x 1.6 x 1.0mm. Current margin is comfortable, since the TPS61099's 0.8A
minimum switch limit bounds peak inductor current well under Isat.

Also found: Taiyo Yuden has renamed this part to LSANB2016KKT2R2M /
LLANB2016KKT2R2M. LCSC still stocks the old code so v2 is unaffected, but
the successors are the direct replacement if C92923 disappears.

Still missing is the land-pattern drawing; LCSC's PDF endpoint serves a bot
page, so it needs fetching by hand. check_parts.py keeps flagging it.

gitignore: added KiCad per-user state (*.kicad_prl), auto-backups and the
VSCode Local History snapshots, and untracked the .kicad_prl already
committed. Design files are untouched and remain tracked.

Co-Authored-By: Claude Opus 5 (1M context) <noreply@anthropic.com>
Parts:
- BT1: footprint pcb_v2:BatteryPads_2x -> pcb:BatteryPads_2x
- L1: footprint pcb_v2:L_MAKK2016T_2.0x1.6mm -> pcb:L_MAKK2016T_2.0x1.6mm
- U1: footprint pcb_v2:ESP32-C3-MINI-1 -> pcb:ESP32-C3-MINI-1
Changed lines of the file:
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@@
       (effects (font (size 1.27 1.27)))
     )
-    (property "Footprint" "pcb_v2:BatteryPads_2x" (at 284.48 55.88 0)
+    (property "Footprint" "pcb:BatteryPads_2x" (at 284.48 55.88 0)
       (effects (font (size 1.27 1.27)) (hide yes))
     )
@@
       (effects (font (size 1.27 1.27)))
     )
-    (property "Footprint" "pcb_v2:L_MAKK2016T_2.0x1.6mm" (at 480.06 40.64 0)
+    (property "Footprint" "pcb:L_MAKK2016T_2.0x1.6mm" (at 480.06 40.64 0)
       (effects (font (size 1.27 1.27)) (hide yes))
     )
@@
       (effects (font (size 1.27 1.27)))
     )
-    (property "Footprint" "pcb_v2:ESP32-C3-MINI-1" (at 109.22 200.66 0)
-      (effects (font (size 1.27 1.27)) (hide yes))
-    )
+    (property "Footprint" "pcb:ESP32-C3-MINI-1" (at 109.22 200.66 0)
+      (effects (font (size 1.27 1.27)) (hide yes))
+    )
