File: pcb/wearable_v2.kicad_sch (KiCad schematic)
At the start: 64 parts, among them J1 TYPE-C-31-M-12, Q1 AO3401A, U1 ESP32-C3-MINI-1-N4, U10 SHT40-AD1B-R3, U2 USBLC6-2SC6, U3 TP4054-42-SOT25R, U4 ME6211C33M5G-N, U5 XC6206P182MR, U6 TPS61099DRVR, U7 MAX30101EFD+T, U8 TMP117AIDRVR, U9 LSM6DS3TR-C

Commit message: again
Parts:
- C1, C15: MPN (none) -> CL10A475KO8NNNC
- C10, C14, C3, C4, C5, C6: MPN (none) -> CL05A105KA5NQNC
- C11, C7, C8, C9: MPN (none) -> CL10A106KP8NNNC
- C12, C13, C16, C17, C18, C19, C2, C20: MPN (none) -> CL05B104KO5NNNC
- D1: MPN (none) -> SS14
- J1: MPN (none) -> TYPE-C-31-M-12
- L1: MPN (none) -> MAKK2016T2R2M
- Q1: MPN (none) -> AO3401A
- R1, R2: MPN (none) -> 0402WGF5101TCE
- R10: MPN (none) -> 0402WGF2703TCE
- R11, R6: MPN (none) -> 0402WGF1003TCE
- R12, R13, R14, R15, R5: MPN (none) -> 0402WGF1002TCE
- R16, R17: MPN (none) -> 0402WGF4701TCE
- R3, R4: MPN (none) -> 0402WGF220JTCE
- R7, R8, R9: MPN (none) -> 0402WGF1004TCE
- U1: MPN (none) -> ESP32-C3-MINI-1-N4
- U10: MPN (none) -> SHT40-AD1B-R3
- U2: MPN (none) -> USBLC6-2SC6
- U3: MPN (none) -> TP4054-42-SOT25R
- U4: MPN (none) -> ME6211C33M5G-N
- U5: MPN (none) -> XC6206P182MR
- U6: MPN (none) -> TPS61099DRVR
- U7: MPN (none) -> MAX30101EFD+T
- U8: MPN (none) -> TMP117AIDRVR
- U9: MPN (none) -> LSM6DS3TR-C
Connections:
- net VSYS: now also U4.1 (V_{IN})
