File: pcb/wearable_v2.kicad_sch (KiCad schematic)
At the start: 64 parts, among them J1 TYPE-C-31-M-12, Q1 AO3401A, U1 ESP32-C3-MINI-1-N4, U10 SHT40-AD1B-R3, U2 USBLC6-2SC6, U3 TP4054-42-SOT25R, U4 ME6211C33M5G-N, U5 XC6206P182MR, U6 TPS61099DRVR, U7 MAX30101EFD+T, U8 TMP117AIDRVR, U9 LSM6DS3TR-C

Commit message: Checkpoint: R10 249k, battery closed, docs reflect verified state
Design change (user-approved):
- R10 270k -> 249k (0402WGF2493TCE / C11425) in schematic and PCB. Value,
  MPN and LCSC only; netlist untouched. Moves the 4V7 worst-case low corner
  from 4.470 V to 4.770 V against the MAX30101's 4.5 V green VLED+ minimum.
- KiCad F8 deliberately not run; property fields patched directly to avoid
  the documented KiCad 10.0.5 stale-U4-pad hazard.
- Re-verified: ERC 2 known warnings, DRC 5 known-acceptable / 0 unconnected,
  parity 0 issues, analyze_pcb.py 51 findings (2/18/31) — all identical to
  the accepted 2026-09-17 baseline.
- Fabrication package regenerated and revalidated 15/15 PASS. Gerber/drill
  ZIP unchanged (R10's value is on F.Fab only, not in the gerber set).
  Caught and fixed a stale wearable_v2_pcba_bom_cpl.zip.

Analysis:
- Desk power/thermal budget: ME6211 dropout and thermal, 3V3 rail under BLE
  TX. Produces a firmware constraint to cap BLE TX at 0 dBm.
- ngspice behavioral simulation of the TPS61099 4V7 boost
  (pcb/analysis/tps61099_4v7_boost.cir). Dynamics are not a risk: a 51 mA
  green LED pulse moves the rail 4 mV. The DC tolerance stack was the only
  failure mode, now fixed by the R10 change.

Battery — closed, final:
- EEMB LP502030-PCM already in hand is the cell for v2. EEMB's own cell
  specification states 250 mA maximum charge; the planned 100 mA is 0.4 C.
  Not to be re-sourced or re-opened.

Documentation:
- New "SETTLED — do not re-verify, do not re-open" section in pcb/README.md
  recording closed checks, the battery decision and the settled JLCPCB
  settings, so future sessions stop re-deriving them.
- Rewrote Current state, Next actions and the stale "Verification NOT done"
  section; flagged the two superseded append-only log rows.
- Synced CLAUDE.md, V2_BOM.md, V2_HARDWARE_AUDIT.md, enclosure/README.md and
  the fabrication README.

Nothing is bench-measured, peer-reviewed or ordered. No order is authorized.

Co-Authored-By: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
Parts:
- R10: value 270k -> 249k; LCSC C25770 -> C11425; MPN 0402WGF2703TCE -> 0402WGF2493TCE
Other:
- note added: "VOUT = 1.0 V x (1M + 249k) / 249k = 5.016 V nominal."
- note removed: "VOUT = 1.0 V x (1M + 270k) / 270k = 4.704 V nominal."
Changed lines of the file:
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@@
 		)
 	)
-	(text "VOUT = 1.0 V x (1M + 270k) / 270k = 4.704 V nominal."
+	(text "VOUT = 1.0 V x (1M + 249k) / 249k = 5.016 V nominal."
 		(exclude_from_sim no)
 		(at 457 116 0)
@@
 			)
 		)
-		(property "Value" "270k"
+		(property "Value" "249k"
 			(at 480.06 102.87 0)
 			(show_name no)
@@
 			)
 		)
-		(property "MPN" "0402WGF2703TCE"
+		(property "MPN" "0402WGF2493TCE"
 			(at 480.06 101.6 0)
 			(hide yes)
@@
 			)
 		)
-		(property "LCSC" "C25770"
+		(property "LCSC" "C11425"
 			(at 480.06 101.6 0)
 			(hide yes)
