File: pcb/wearable_v2.kicad_pcb (KiCad board)
At the start: 4 copper layers, 64 parts, among them J1 TYPE-C-31-M-12, Q1 AO3401A, U1 ESP32-C3-MINI-1-N4, U10 SHT40-AD1B-R3, U2 USBLC6-2SC6, U3 TP4054-42-SOT25R, U4 ME6211C33M5G-N, U5 XC6206P182MR, U6 TPS61099DRVR, U7 MAX30101EFD+T, U8 TMP117AIDRVR, U9 LSM6DS3TR-C

Commit message: orchestrator/subagent architecture, BACtrack comp analysis
Parts:
- C13, C14, C15, C17, U7, U8: moved to B.Cu
- moved C12 36.7 mm to (63.8, 108.0)
- moved Q1 36.1 mm to (65.0, 132.4)
- moved C4 35.0 mm to (63.8, 109.3)
- moved BT1 34.1 mm to (65.4, 142.0), turned to 180 degrees
- moved C10 32.5 mm to (63.8, 113.2)
- moved C19 28.8 mm to (67.6, 124.0)
- moved C18 28.6 mm to (67.6, 122.6)
- moved C2 28.2 mm to (63.8, 117.1)
- moved D1 28.1 mm to (65.0, 136.0)
- moved C17 27.6 mm to (67.5, 133.5), turned to 180 degrees
- moved TP6 26.2 mm to (61.5, 130.0)
- moved C20 25.5 mm to (70.5, 143.2)
- moved TP7 25.0 mm to (61.3, 112.0)
- moved R12 24.7 mm to (63.8, 111.9)
- moved U5 23.8 mm to (78.0, 132.6)
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Connections:
- U4 pad 1: unconnected-(U4-V_{IN}-Pad1) -> VSYS
Routing:
- net GND: track 0.00 -> 219.3 mm, vias 0 -> 2
- net 3V3: track 0.00 -> 115.9 mm, vias 0 -> 6
- net /SDA: track 0.00 -> 58.8 mm, vias 0 -> 4
- net /USB_DP: track 0.00 -> 51.7 mm, vias 0 -> 2
- net VSYS: track 0.00 -> 47.7 mm, vias 0 -> 2
- net /USB_DM_CON: track 0.00 -> 38.5 mm, vias 0 -> 2
- net BAT+: track 0.00 -> 34.9 mm, vias 0 -> 2
- net /SCL: track 0.00 -> 34.3 mm, vias 0 -> 3
- net 4V7: track 0.00 -> 34.0 mm, vias 0 -> 4
- net VBUS: track 0.00 -> 30.7 mm, vias 0 -> 3
- net /USB_DM: track 0.00 -> 28.0 mm, vias 0 -> 2
- net 1V8: track 0.00 -> 25.0 mm, vias 0 -> 2
- net /USB_DP_CON: track 0.00 -> 12.8 mm, vias 0 -> 2
- net /CC2: track 0.00 -> 12.5 mm, vias 0 -> 2
- net /BAT_SENSE: track 0.00 -> 10.9 mm, vias 0 -> 2
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Other:
- board outline added: 24 x 46 mm
- board text added: "LiPo 402030 30x20 CELL BODY (on top)"
